Commit message: Scanner mount

File: kortex_description/arms/gen3/6dof/urdf/gen3_macro.xacro (robot description, xacro)
@@ -353,4 +353,26 @@
         xyz="0 0 0" />
     </joint>
+    <joint name="${prefix}kinova_mount_joint" type="fixed">
+      <origin xyz="0 0 -0.03" rpy="0 ${PI} 0" />
+      <parent link="${prefix}end_effector_link" />
+      <child link="${prefix}kinova_mount_link" />
+    </joint>
+    <link name="${prefix}kinova_mount_link">
+      <visual>
+        <origin xyz="0 0 -0.03" rpy="0 0 0" />
+        <geometry>
+          <mesh filename="file://$(find kortex_description)/arms/gen3/meshes/kinova_mount.stl" scale="0.001 0.001 0.001" />
+        </geometry>
+        <material name="">
+          <color rgba="0.75294 0.75294 0.75294 1" />
+        </material>
+      </visual>
+      <collision>
+        <origin xyz="0 0 -0.03" rpy="0 0 0" />
+        <geometry>
+          <mesh filename="file://$(find kortex_description)/arms/gen3/meshes/kinova_mount.stl" scale="0.001 0.001 0.001" />
+        </geometry>
+      </collision>
+    </link>
     <!-- TODO(destogl) this probably collides with camera URDF -->
     <xacro:if value="${vision}">

File: kortex_description/arms/gen3/7dof/urdf/gen3_macro.xacro (robot description, xacro)
@@ -447,4 +447,26 @@
         xyz="0 0 0" />
     </joint>
+    <joint name="${prefix}kinova_mount_joint" type="fixed">
+      <origin xyz="0 0 0" rpy="0 ${PI} 0" />
+      <parent link="${prefix}end_effector_link" />
+      <child link="${prefix}kinova_mount_link" />
+    </joint>
+    <link name="${prefix}kinova_mount_link">
+      <visual>
+        <origin xyz="0 0 -0.03" rpy="0 0 0" />
+        <geometry>
+          <mesh filename="file://$(find kortex_description)/arms/gen3/meshes/kinova_mount.stl" scale="0.001 0.001 0.001" />
+        </geometry>
+        <material name="">
+          <color rgba="0.75294 0.75294 0.75294 1" />
+        </material>
+      </visual>
+      <collision>
+        <origin xyz="0 0 -0.03" rpy="0 0 0" />
+        <geometry>
+          <mesh filename="file://$(find kortex_description)/arms/gen3/meshes/kinova_mount.stl" scale="0.001 0.001 0.001" />
+        </geometry>
+      </collision>
+    </link>
     <xacro:if value="${vision}">
       <!-- sim camera needs to be rotated which might not apply to built in vision module -->

Commit message: Add reference to clarius_description

File: kortex_description/arms/gen3/6dof/urdf/gen3_macro.xacro (robot description, xacro)
@@ -4,4 +4,5 @@
   <xacro:property name="last_arm_link" value="end_effector_link"/>
   <xacro:property name="PI" value="3.1415926535897931"/>
+  <xacro:include filename="$(find clarius_description)/urdf/clarius_macro.xacro" />
   <xacro:macro name="load_arm" params="
     parent
@@ -375,4 +376,7 @@
       </collision>
     </link>
+    <xacro:load_clarius parent="${prefix}kinova_mount_link" prefix="${prefix}">
+      <origin xyz="0 0 -0.05" rpy="0 ${PI} ${PI/2}" />
+    </xacro:load_clarius>
     <!-- TODO(destogl) this probably collides with camera URDF -->
     <xacro:if value="${vision}">

File: kortex_description/arms/gen3/7dof/urdf/gen3_macro.xacro (robot description, xacro)
@@ -4,4 +4,5 @@
   <xacro:property name="last_arm_link" value="end_effector_link"/>
   <xacro:property name="PI" value="3.1415926535897931"/>
+  <xacro:include filename="$(find clarius_description)/urdf/clarius_macro.xacro" />
   <xacro:macro name="load_arm" params="
     parent
@@ -469,4 +470,7 @@
       </collision>
     </link>
+    <xacro:load_clarius parent="${prefix}kinova_mount_link" prefix="${prefix}">
+      <origin xyz="0 0 -0.05" rpy="0 ${PI} ${PI/2}" />
+    </xacro:load_clarius>
     <xacro:if value="${vision}">
       <!-- sim camera needs to be rotated which might not apply to built in vision module -->

Commit message: Update mesh to be 8 mm taller and adjust URDFs

File: kortex_description/arms/gen3/6dof/urdf/gen3_macro.xacro (robot description, xacro)
@@ -355,5 +355,5 @@
     </joint>
     <joint name="${prefix}kinova_mount_joint" type="fixed">
-      <origin xyz="0 0 -0.03" rpy="0 ${PI} 0" />
+      <origin xyz="0 0 0" rpy="0 ${PI} 0" />
       <parent link="${prefix}end_effector_link" />
       <child link="${prefix}kinova_mount_link" />
@@ -361,5 +361,5 @@
     <link name="${prefix}kinova_mount_link">
       <visual>
-        <origin xyz="0 0 -0.03" rpy="0 0 0" />
+        <origin xyz="0 0 -0.038" rpy="0 0 0" />
         <geometry>
           <mesh filename="file://$(find kortex_description)/arms/gen3/meshes/kinova_mount.stl" scale="0.001 0.001 0.001" />
@@ -370,5 +370,5 @@
       </visual>
       <collision>
-        <origin xyz="0 0 -0.03" rpy="0 0 0" />
+        <origin xyz="0 0 -0.038" rpy="0 0 0" />
         <geometry>
           <mesh filename="file://$(find kortex_description)/arms/gen3/meshes/kinova_mount.stl" scale="0.001 0.001 0.001" />
@@ -377,5 +377,5 @@
     </link>
     <xacro:load_clarius parent="${prefix}kinova_mount_link" prefix="${prefix}">
-      <origin xyz="0 0 -0.05" rpy="0 ${PI} ${PI/2}" />
+      <origin xyz="0 0 -0.058" rpy="0 ${PI} ${PI/2}" />
     </xacro:load_clarius>
     <!-- TODO(destogl) this probably collides with camera URDF -->

File: kortex_description/arms/gen3/7dof/urdf/gen3_macro.xacro (robot description, xacro)
@@ -455,5 +455,5 @@
     <link name="${prefix}kinova_mount_link">
       <visual>
-        <origin xyz="0 0 -0.03" rpy="0 0 0" />
+        <origin xyz="0 0 -0.038" rpy="0 0 0" />
         <geometry>
           <mesh filename="file://$(find kortex_description)/arms/gen3/meshes/kinova_mount.stl" scale="0.001 0.001 0.001" />
@@ -464,5 +464,5 @@
       </visual>
       <collision>
-        <origin xyz="0 0 -0.03" rpy="0 0 0" />
+        <origin xyz="0 0 -0.038" rpy="0 0 0" />
         <geometry>
           <mesh filename="file://$(find kortex_description)/arms/gen3/meshes/kinova_mount.stl" scale="0.001 0.001 0.001" />
@@ -471,5 +471,5 @@
     </link>
     <xacro:load_clarius parent="${prefix}kinova_mount_link" prefix="${prefix}">
-      <origin xyz="0 0 -0.05" rpy="0 ${PI} ${PI/2}" />
+      <origin xyz="0 0 -0.058" rpy="0 ${PI} ${PI/2}" />
     </xacro:load_clarius>
     <xacro:if value="${vision}">

Commit message: Updated the scanner mount to match the new design

File: kortex_description/arms/gen3/6dof/urdf/gen3_macro.xacro (robot description, xacro)
@@ -355,5 +355,5 @@
     </joint>
     <joint name="${prefix}kinova_mount_joint" type="fixed">
-      <origin xyz="0 0 0" rpy="0 ${PI} 0" />
+      <origin xyz="0 0 0.003" rpy="0 ${PI} 0" />
       <parent link="${prefix}end_effector_link" />
       <child link="${prefix}kinova_mount_link" />
@@ -361,21 +361,21 @@
     <link name="${prefix}kinova_mount_link">
       <visual>
-        <origin xyz="0 0 -0.038" rpy="0 0 0" />
-        <geometry>
-          <mesh filename="file://$(find kortex_description)/arms/gen3/meshes/kinova_mount.stl" scale="0.001 0.001 0.001" />
-        </geometry>
-        <material name="">
-          <color rgba="0.75294 0.75294 0.75294 1" />
-        </material>
-      </visual>
-      <collision>
-        <origin xyz="0 0 -0.038" rpy="0 0 0" />
-        <geometry>
-          <mesh filename="file://$(find kortex_description)/arms/gen3/meshes/kinova_mount.stl" scale="0.001 0.001 0.001" />
+        <origin xyz="0 0 0" rpy="-1.5708 0 0" />
+        <geometry>
+          <mesh filename="file://$(find kortex_description)/arms/gen3/meshes/kinova_mount.stl" scale="1 1 1" />
+        </geometry>
+        <material name="">
+          <color rgba="0.75294 0.75294 0.75294 1" />
+        </material>
+      </visual>
+      <collision>
+        <origin xyz="0 0 0" rpy="-1.5708 0 0" />
+        <geometry>
+          <mesh filename="file://$(find kortex_description)/arms/gen3/meshes/kinova_mount.stl" scale="1 1 1" />
         </geometry>
       </collision>
     </link>
     <xacro:load_clarius parent="${prefix}kinova_mount_link" prefix="${prefix}">
-      <origin xyz="0 0 -0.058" rpy="0 ${PI} ${PI/2}" />
+      <origin xyz="0 0 -0.115" rpy="${PI/2} ${PI} ${PI}" />
     </xacro:load_clarius>
     <!-- TODO(destogl) this probably collides with camera URDF -->

File: kortex_description/arms/gen3/7dof/urdf/gen3_macro.xacro (robot description, xacro)
@@ -449,5 +449,5 @@
     </joint>
     <joint name="${prefix}kinova_mount_joint" type="fixed">
-      <origin xyz="0 0 0" rpy="0 ${PI} 0" />
+      <origin xyz="0 0 0.003" rpy="0 ${PI} 0" />
       <parent link="${prefix}end_effector_link" />
       <child link="${prefix}kinova_mount_link" />
@@ -455,21 +455,21 @@
     <link name="${prefix}kinova_mount_link">
       <visual>
-        <origin xyz="0 0 -0.038" rpy="0 0 0" />
-        <geometry>
-          <mesh filename="file://$(find kortex_description)/arms/gen3/meshes/kinova_mount.stl" scale="0.001 0.001 0.001" />
-        </geometry>
-        <material name="">
-          <color rgba="0.75294 0.75294 0.75294 1" />
-        </material>
-      </visual>
-      <collision>
-        <origin xyz="0 0 -0.038" rpy="0 0 0" />
-        <geometry>
-          <mesh filename="file://$(find kortex_description)/arms/gen3/meshes/kinova_mount.stl" scale="0.001 0.001 0.001" />
+        <origin xyz="0 0 0" rpy="-1.5708 0 0" />
+        <geometry>
+          <mesh filename="file://$(find kortex_description)/arms/gen3/meshes/kinova_mount.stl" scale="1 1 1" />
+        </geometry>
+        <material name="">
+          <color rgba="0.75294 0.75294 0.75294 1" />
+        </material>
+      </visual>
+      <collision>
+        <origin xyz="0 0 0" rpy="-1.5708 0 0" />
+        <geometry>
+          <mesh filename="file://$(find kortex_description)/arms/gen3/meshes/kinova_mount.stl" scale="1 1 1" />
         </geometry>
       </collision>
     </link>
     <xacro:load_clarius parent="${prefix}kinova_mount_link" prefix="${prefix}">
-      <origin xyz="0 0 -0.058" rpy="0 ${PI} ${PI/2}" />
+      <origin xyz="0 0 -0.115" rpy="${PI/2} ${PI} ${PI}" />
     </xacro:load_clarius>
     <xacro:if value="${vision}">
