Commit message: Fixed torque-sign correction

File: kortex_description/grippers/robotiq_2f_85/urdf/robotiq_2f_85_macro.xacro (robot description, xacro)
@@ -7,4 +7,5 @@
     fake_sensor_commands:=false
     sim_ignition:=false
+    sim_mujoco:=false
     sim_isaac:=false
     isaac_joint_commands:=/isaac_joint_commands
@@ -16,5 +17,5 @@
     <!-- Hardware talks directly to the gripper so we don't need ros2_control unless we are simulating -->
     <xacro:property name="include_ros2_control" value="false"/>
-    <xacro:if value="${sim_ignition or sim_isaac or use_fake_hardware or not use_internal_bus_gripper_comm}">
+    <xacro:if value="${not sim_mujoco and (sim_ignition or sim_isaac or use_fake_hardware or not use_internal_bus_gripper_comm)}">
       <xacro:property name="include_ros2_control" value="true"/>
     </xacro:if>
@@ -31,6 +32,16 @@
         isaac_joint_commands="${isaac_joint_commands}"
         isaac_joint_states="${isaac_joint_states}">
+        <!-- Match view_robot.launch.py: the gripper mounting plane is
+             coincident with the arm end-effector flange. -->
         <origin xyz="0 0 0" rpy="0 0 0" />
     </xacro:robotiq_gripper>
+    <!-- The requested 0.12 m transform is the gripper tool point, not an
+         offset between the flange and the gripper body. -->
+    <link name="${prefix}tool_frame"/>
+    <joint name="${prefix}tool_frame_joint" type="fixed">
+      <origin xyz="0 0 0.12" rpy="0 0 0" />
+      <parent link="${prefix}robotiq_85_base_link" />
+      <child link="${prefix}tool_frame" />
+    </joint>
   </xacro:macro>
 </robot>

File: kortex_description/robots/kortex_robot.xacro (robot description, xacro)
@@ -118,4 +118,5 @@
         fake_sensor_commands="${fake_sensor_commands}"
         sim_ignition="${sim_ignition}"
+        sim_mujoco="${sim_mujoco}"
         sim_isaac="${sim_isaac}"
         isaac_joint_commands="${isaac_joint_commands}"
