Commit message: Added admittance controller and verified in Rviz2

File: kortex_description/arms/gen3/7dof/urdf/gen3_macro.xacro (robot description, xacro)
@@ -4,5 +4,4 @@
   <xacro:property name="last_arm_link" value="end_effector_link"/>
   <xacro:property name="PI" value="3.1415926535897931"/>
-  <xacro:include filename="$(find clarius_description)/urdf/clarius_macro.xacro" />
   <xacro:macro name="load_arm" params="
     parent
@@ -22,4 +21,20 @@
     gripper_max_velocity:=100.0
     gripper_max_force:=100.0
+    wrench_filter_coefficient:=0.05
+    wrench_force_deadband:=2.0
+    wrench_torque_deadband:=0.2
+    wrench_force_limit:=40.0
+    wrench_torque_limit:=8.0
+    wrench_force_stop_threshold:=80.0
+    wrench_torque_stop_threshold:=15.0
+    wrench_bias_force_x:=0.0
+    wrench_bias_force_y:=0.0
+    wrench_bias_force_z:=0.0
+    wrench_bias_torque_x:=0.0
+    wrench_bias_torque_y:=0.0
+    wrench_bias_torque_z:=0.0
+    feedback_timeout:=0.1
+    max_joint_command_velocity:=0.25
+    joint_limit_margin:=0.02
     use_fake_hardware:=false
     fake_sensor_commands:=false
@@ -30,4 +45,5 @@
     isaac_joint_states:=/isaac_joint_states
     use_external_cable:=false
+    include_clarius:=true
     initial_positions:=${dict(joint_1=0.0,joint_2=0.0,joint_3=0.0,joint_4=0.0,joint_5=0.0,joint_6=0.0,joint_7=0.0)}
     moveit_active:=false">
@@ -56,5 +72,21 @@
       gripper_max_velocity="${gripper_max_velocity}"
       gripper_max_force="${gripper_max_force}"
-      gripper_joint_name="${gripper_joint_name}"/>
+      gripper_joint_name="${gripper_joint_name}"
+      wrench_filter_coefficient="${wrench_filter_coefficient}"
+      wrench_force_deadband="${wrench_force_deadband}"
+      wrench_torque_deadband="${wrench_torque_deadband}"
+      wrench_force_limit="${wrench_force_limit}"
+      wrench_torque_limit="${wrench_torque_limit}"
+      wrench_force_stop_threshold="${wrench_force_stop_threshold}"
+      wrench_torque_stop_threshold="${wrench_torque_stop_threshold}"
+      wrench_bias_force_x="${wrench_bias_force_x}"
+      wrench_bias_force_y="${wrench_bias_force_y}"
+      wrench_bias_force_z="${wrench_bias_force_z}"
+      wrench_bias_torque_x="${wrench_bias_torque_x}"
+      wrench_bias_torque_y="${wrench_bias_torque_y}"
+      wrench_bias_torque_z="${wrench_bias_torque_z}"
+      feedback_timeout="${feedback_timeout}"
+      max_joint_command_velocity="${max_joint_command_velocity}"
+      joint_limit_margin="${joint_limit_margin}"/>
     <joint name="${prefix}base_joint" type="fixed">
       <xacro:insert_block name="origin" />
@@ -448,29 +480,32 @@
         xyz="0 0 0" />
     </joint>
-    <joint name="${prefix}kinova_mount_joint" type="fixed">
-      <origin xyz="0 0 0.003" rpy="0 ${PI} 0" />
-      <parent link="${prefix}end_effector_link" />
-      <child link="${prefix}kinova_mount_link" />
-    </joint>
-    <link name="${prefix}kinova_mount_link">
-      <visual>
-        <origin xyz="0 0 0" rpy="-1.5708 0 0" />
-        <geometry>
-          <mesh filename="file://$(find kortex_description)/arms/gen3/meshes/kinova_mount.stl" scale="1 1 1" />
-        </geometry>
-        <material name="">
-          <color rgba="0.75294 0.75294 0.75294 1" />
-        </material>
-      </visual>
-      <collision>
-        <origin xyz="0 0 0" rpy="-1.5708 0 0" />
-        <geometry>
-          <mesh filename="file://$(find kortex_description)/arms/gen3/meshes/kinova_mount.stl" scale="1 1 1" />
-        </geometry>
-      </collision>
-    </link>
-    <xacro:load_clarius parent="${prefix}kinova_mount_link" prefix="${prefix}">
-      <origin xyz="0 0 -0.115" rpy="${PI/2} ${PI} ${PI}" />
-    </xacro:load_clarius>
+    <xacro:if value="${include_clarius}">
+      <xacro:include filename="$(find clarius_description)/urdf/clarius_macro.xacro" />
+      <joint name="${prefix}kinova_mount_joint" type="fixed">
+        <origin xyz="0 0 0.003" rpy="0 ${PI} 0" />
+        <parent link="${prefix}end_effector_link" />
+        <child link="${prefix}kinova_mount_link" />
+      </joint>
+      <link name="${prefix}kinova_mount_link">
+        <visual>
+          <origin xyz="0 0 0" rpy="-1.5708 0 0" />
+          <geometry>
+            <mesh filename="file://$(find kortex_description)/arms/gen3/meshes/kinova_mount.stl" scale="1 1 1" />
+          </geometry>
+          <material name="">
+            <color rgba="0.75294 0.75294 0.75294 1" />
+          </material>
+        </visual>
+        <collision>
+          <origin xyz="0 0 0" rpy="-1.5708 0 0" />
+          <geometry>
+            <mesh filename="file://$(find kortex_description)/arms/gen3/meshes/kinova_mount.stl" scale="1 1 1" />
+          </geometry>
+        </collision>
+      </link>
+      <xacro:load_clarius parent="${prefix}kinova_mount_link" prefix="${prefix}">
+        <origin xyz="0 0 -0.115" rpy="${PI/2} ${PI} ${PI}" />
+      </xacro:load_clarius>
+    </xacro:if>
     <xacro:if value="${vision}">
       <!-- sim camera needs to be rotated which might not apply to built in vision module -->

File: kortex_description/arms/gen3/7dof/urdf/kortex.ros2_control.xacro (robot description, xacro)
@@ -24,4 +24,20 @@
     gripper_max_velocity:=100.0
     gripper_max_force:=100.0
+    wrench_filter_coefficient:=0.05
+    wrench_force_deadband:=2.0
+    wrench_torque_deadband:=0.2
+    wrench_force_limit:=40.0
+    wrench_torque_limit:=8.0
+    wrench_force_stop_threshold:=80.0
+    wrench_torque_stop_threshold:=15.0
+    wrench_bias_force_x:=0.0
+    wrench_bias_force_y:=0.0
+    wrench_bias_force_z:=0.0
+    wrench_bias_torque_x:=0.0
+    wrench_bias_torque_y:=0.0
+    wrench_bias_torque_z:=0.0
+    feedback_timeout:=0.1
+    max_joint_command_velocity:=0.25
+    joint_limit_margin:=0.02
     moveit_active:=false">
     <ros2_control name="${name}" type="system">
@@ -40,5 +56,5 @@
         <xacro:if value="${use_fake_hardware}">
           <plugin>mock_components/GenericSystem</plugin>
-          <param name="fake_sensor_commands">${fake_sensor_commands}</param>
+          <param name="mock_sensor_commands">${fake_sensor_commands}</param>
           <param name="state_following_offset">0.0</param>
         </xacro:if>
@@ -58,4 +74,20 @@
           <param name="gripper_max_velocity">${gripper_max_velocity}</param>
           <param name="gripper_max_force">${gripper_max_force}</param>
+          <param name="wrench_filter_coefficient">${wrench_filter_coefficient}</param>
+          <param name="wrench_force_deadband">${wrench_force_deadband}</param>
+          <param name="wrench_torque_deadband">${wrench_torque_deadband}</param>
+          <param name="wrench_force_limit">${wrench_force_limit}</param>
+          <param name="wrench_torque_limit">${wrench_torque_limit}</param>
+          <param name="wrench_force_stop_threshold">${wrench_force_stop_threshold}</param>
+          <param name="wrench_torque_stop_threshold">${wrench_torque_stop_threshold}</param>
+          <param name="wrench_bias_force_x">${wrench_bias_force_x}</param>
+          <param name="wrench_bias_force_y">${wrench_bias_force_y}</param>
+          <param name="wrench_bias_force_z">${wrench_bias_force_z}</param>
+          <param name="wrench_bias_torque_x">${wrench_bias_torque_x}</param>
+          <param name="wrench_bias_torque_y">${wrench_bias_torque_y}</param>
+          <param name="wrench_bias_torque_z">${wrench_bias_torque_z}</param>
+          <param name="feedback_timeout">${feedback_timeout}</param>
+          <param name="max_joint_command_velocity">${max_joint_command_velocity}</param>
+          <param name="joint_limit_margin">${joint_limit_margin}</param>
         </xacro:unless>
       </hardware>
@@ -137,4 +169,12 @@
         <state_interface name="effort"/>
       </joint>
+      <sensor name="${prefix}tool_external_wrench">
+        <state_interface name="force.x"/>
+        <state_interface name="force.y"/>
+        <state_interface name="force.z"/>
+        <state_interface name="torque.x"/>
+        <state_interface name="torque.y"/>
+        <state_interface name="torque.z"/>
+      </sensor>
       <xacro:unless value="${use_fake_hardware or sim_gazebo or sim_ignition or sim_isaac}">
         <xacro:if value="${use_internal_bus_gripper_comm}">

File: kortex_description/robots/gen3.xacro (robot description, xacro)
@@ -16,4 +16,20 @@
     <xacro:arg name="gripper_max_velocity" default="100.0" />
     <xacro:arg name="gripper_max_force" default="100.0" />
+    <xacro:arg name="wrench_filter_coefficient" default="0.05" />
+    <xacro:arg name="wrench_force_deadband" default="2.0" />
+    <xacro:arg name="wrench_torque_deadband" default="0.2" />
+    <xacro:arg name="wrench_force_limit" default="40.0" />
+    <xacro:arg name="wrench_torque_limit" default="8.0" />
+    <xacro:arg name="wrench_force_stop_threshold" default="80.0" />
+    <xacro:arg name="wrench_torque_stop_threshold" default="15.0" />
+    <xacro:arg name="wrench_bias_force_x" default="0.0" />
+    <xacro:arg name="wrench_bias_force_y" default="0.0" />
+    <xacro:arg name="wrench_bias_force_z" default="0.0" />
+    <xacro:arg name="wrench_bias_torque_x" default="0.0" />
+    <xacro:arg name="wrench_bias_torque_y" default="0.0" />
+    <xacro:arg name="wrench_bias_torque_z" default="0.0" />
+    <xacro:arg name="feedback_timeout" default="0.1" />
+    <xacro:arg name="max_joint_command_velocity" default="0.25" />
+    <xacro:arg name="joint_limit_margin" default="0.02" />
     <xacro:arg name="sim_gazebo" default="false" />
     <xacro:arg name="sim_ignition" default="false" />
@@ -24,4 +40,5 @@
     <xacro:arg name="use_internal_bus_gripper_comm" default="false" />
     <xacro:arg name="use_external_cable" default="false" />
+    <xacro:arg name="include_clarius" default="true" />
     <xacro:include filename="$(find kortex_description)/robots/kortex_robot.xacro" />
     <!-- initial position for simulations (Mock Hardware, Gazebo, Ignition) -->
@@ -37,4 +54,20 @@
         gripper_max_velocity="$(arg gripper_max_velocity)"
         gripper_max_force="$(arg gripper_max_force)"
+        wrench_filter_coefficient="$(arg wrench_filter_coefficient)"
+        wrench_force_deadband="$(arg wrench_force_deadband)"
+        wrench_torque_deadband="$(arg wrench_torque_deadband)"
+        wrench_force_limit="$(arg wrench_force_limit)"
+        wrench_torque_limit="$(arg wrench_torque_limit)"
+        wrench_force_stop_threshold="$(arg wrench_force_stop_threshold)"
+        wrench_torque_stop_threshold="$(arg wrench_torque_stop_threshold)"
+        wrench_bias_force_x="$(arg wrench_bias_force_x)"
+        wrench_bias_force_y="$(arg wrench_bias_force_y)"
+        wrench_bias_force_z="$(arg wrench_bias_force_z)"
+        wrench_bias_torque_x="$(arg wrench_bias_torque_x)"
+        wrench_bias_torque_y="$(arg wrench_bias_torque_y)"
+        wrench_bias_torque_z="$(arg wrench_bias_torque_z)"
+        feedback_timeout="$(arg feedback_timeout)"
+        max_joint_command_velocity="$(arg max_joint_command_velocity)"
+        joint_limit_margin="$(arg joint_limit_margin)"
         dof="$(arg dof)"
         vision="$(arg vision)"
@@ -54,4 +87,5 @@
         sim_isaac="$(arg sim_isaac)"
         use_external_cable="$(arg use_external_cable)"
+        include_clarius="$(arg include_clarius)"
         initial_positions="${xacro.load_yaml(initial_positions_file)}" >
         <origin xyz="0 0 0" rpy="0 0 0" />  <!-- position robot in the world -->

File: kortex_description/robots/kortex_robot.xacro (robot description, xacro)
@@ -26,7 +26,24 @@
     isaac_joint_states:=/isaac_joint_states
     use_external_cable:=false
+    include_clarius:=true
     initial_positions:=${dict(joint_1=0.0,joint_2=0.0,joint_3=0.0,joint_4=0.0,joint_5=0.0,joint_6=0.0,joint_7=0.0)}
     gripper_max_velocity:=100.0
     gripper_max_force:=100.0
+    wrench_filter_coefficient:=0.05
+    wrench_force_deadband:=2.0
+    wrench_torque_deadband:=0.2
+    wrench_force_limit:=40.0
+    wrench_torque_limit:=8.0
+    wrench_force_stop_threshold:=80.0
+    wrench_torque_stop_threshold:=15.0
+    wrench_bias_force_x:=0.0
+    wrench_bias_force_y:=0.0
+    wrench_bias_force_z:=0.0
+    wrench_bias_torque_x:=0.0
+    wrench_bias_torque_y:=0.0
+    wrench_bias_torque_z:=0.0
+    feedback_timeout:=0.1
+    max_joint_command_velocity:=0.25
+    joint_limit_margin:=0.02
     gripper_com_port:=/dev/ttyUSB0
     moveit_active:=false">
@@ -57,4 +74,21 @@
       gripper_max_velocity="${gripper_max_velocity}"
       gripper_max_force="${gripper_max_force}"
+      include_clarius="${include_clarius}"
+      wrench_filter_coefficient="${wrench_filter_coefficient}"
+      wrench_force_deadband="${wrench_force_deadband}"
+      wrench_torque_deadband="${wrench_torque_deadband}"
+      wrench_force_limit="${wrench_force_limit}"
+      wrench_torque_limit="${wrench_torque_limit}"
+      wrench_force_stop_threshold="${wrench_force_stop_threshold}"
+      wrench_torque_stop_threshold="${wrench_torque_stop_threshold}"
+      wrench_bias_force_x="${wrench_bias_force_x}"
+      wrench_bias_force_y="${wrench_bias_force_y}"
+      wrench_bias_force_z="${wrench_bias_force_z}"
+      wrench_bias_torque_x="${wrench_bias_torque_x}"
+      wrench_bias_torque_y="${wrench_bias_torque_y}"
+      wrench_bias_torque_z="${wrench_bias_torque_z}"
+      feedback_timeout="${feedback_timeout}"
+      max_joint_command_velocity="${max_joint_command_velocity}"
+      joint_limit_margin="${joint_limit_margin}"
       use_external_cable="${use_external_cable}"
       initial_positions="${initial_positions}"

Commit message: Added gracity-holding position servos for all joints

File: kortex_description/arms/gen3/7dof/urdf/gen3_macro.xacro (robot description, xacro)
@@ -91,4 +91,27 @@
       max_joint_command_velocity="${max_joint_command_velocity}"
       joint_limit_margin="${joint_limit_margin}"/>
+    <xacro:if value="${sim_mujoco}">
+      <!--
+        The MuJoCo hardware plugin forwards position commands to these servos.
+        Without an actuator the generated model is passive, so the arm falls as
+        soon as gravity is enabled.  The force ranges match the Gen3 URDF joint
+        effort limits except for the shoulder/elbow, which use 120 Nm so the
+        imported inertial model can hold the all-zero startup pose under gravity.
+      -->
+      <mujoco>
+        <default>
+          <joint damping="2.0"/>
+        </default>
+        <actuator>
+          <position name="position_joint_1" joint="${prefix}joint_1" kp="2000" forcelimited="true" forcerange="-120 120"/>
+          <position name="position_joint_2" joint="${prefix}joint_2" kp="2000" forcelimited="true" forcerange="-120 120"/>
+          <position name="position_joint_3" joint="${prefix}joint_3" kp="2000" forcelimited="true" forcerange="-120 120"/>
+          <position name="position_joint_4" joint="${prefix}joint_4" kp="2000" forcelimited="true" forcerange="-120 120"/>
+          <position name="position_joint_5" joint="${prefix}joint_5" kp="250" forcelimited="true" forcerange="-9 9"/>
+          <position name="position_joint_6" joint="${prefix}joint_6" kp="250" forcelimited="true" forcerange="-9 9"/>
+          <position name="position_joint_7" joint="${prefix}joint_7" kp="250" forcelimited="true" forcerange="-9 9"/>
+        </actuator>
+      </mujoco>
+    </xacro:if>
     <joint name="${prefix}base_joint" type="fixed">
       <xacro:insert_block name="origin" />

Commit message: Added nullspace posture restoration to prevent drifts

File: kortex_description/arms/gen3/7dof/urdf/gen3_macro.xacro (robot description, xacro)
@@ -421,4 +421,5 @@
     <link name="${prefix}bracelet_link">
       <inertial>
+        <!-- <origin xyz="-0.000281 -0.011402 -0.029798" rpy="0 0 0" /> -->
         <origin xyz="0.000281 0.011402 -0.029798" rpy="0 0 0" />
         <mass value="0.5" />
